File: hardware/MCP73831.sch (KiCad schematic (older format))
At the start: 14 parts

Commit message: update,
Parts:
- removed C?: CP47uf,16V, Capacitor_SMD:CP_Elec_5x5.3, symbol taobao-cp:CP47uf,16V
- added C1: C106,0805, Capacitor_SMD:C_0805_2012Metric_Pad1.15x1.40mm_HandSolder, symbol taobao-c:C106,0805
- F1: renamed from F?; value Fuse_Small -> Fuse_Small,0805; footprint (none) -> Resistor_SMD:R_0805_2012Metric_Pad1.15x1.40mm_HandSolder
- gave numbers to parts that had none: 12
Connections:
- wire segments 41 -> 43
- no-connect marks 0 -> 3
Changed lines of the file:
@@
 EESchema Schematic File Version 4
+LIBS:MCP73831-cache
 EELAYER 29 0
 EELAYER END
 $Descr User 8500 5500
 encoding utf-8
-Sheet 1 2
+Sheet 1 1
 Title ""
 Date ""
@@
 EndData
 $EndBitmap
-$Sheet
-S 1250 750  950  600
-U 5CF53CAE
-F0 "Sheet5CF53CAD" 50
-F1 "LM2940.sch" 50
-F2 "Vinput" I L 1250 900 50
-F3 "5v_reg_output" O R 2200 1100 50
-$EndSheet
-$Comp
-L taobao-components:MCP73837_MSOP10 U?
+$Comp
+L taobao-components:MCP73837_MSOP10 U2
 U 1 1 5CF6CF79
 P 4750 2400
-F 0 "U?" H 4750 3400 50  0000 C CNN
+F 0 "U2" H 4750 3400 50  0000 C CNN
 F 1 "MCP73837_MSOP10" H 4750 3300 50  0000 C CNN
 F 2 "footprint-lib:MCP73837_MSOP10" H 4775 950 50  0001 C CNN
@@
 $EndComp
 $Comp
-L power:GND #PWR?
+L power:GND #PWR0101
 U 1 1 5CF6D476
 P 4550 3350
-F 0 "#PWR?" H 4550 3100 50  0001 C CNN
+F 0 "#PWR0101" H 4550 3100 50  0001 C CNN
 F 1 "GND" H 4600 3150 50  0000 C CNN
 F 2 "" H 4550 3350 50  0001 C CNN
@@
 	4550 3300 4550 3350
 $Comp
-L power:GND #PWR?
+L power:GND #PWR0102
 U 1 1 5CF6D755
 P 5000 3350
-F 0 "#PWR?" H 5000 3100 50  0001 C CNN
+F 0 "#PWR0102" H 5000 3100 50  0001 C CNN
 F 1 "GND" H 5050 3150 50  0000 C CNN
 F 2 "" H 5000 3350 50  0001 C CNN
@@
 	5000 3300 5000 3350
 $Comp
-L taobao-d:D_1N4148_T4 D?
+L taobao-d:D_1N4148_T4 D1
 U 1 1 5CF71D07
 P 2550 1800
-F 0 "D?" H 2550 1550 50  0000 C CNN
+F 0 "D1" H 2550 1550 50  0000 C CNN
 F 1 "D_1N4148_T4" H 2550 1650 50  0000 C CNN
 F 2 "Diode_SMD:D_SOD-123" V 2550 1800 50  0001 C CNN
@@
 $EndComp
 $Comp
-L taobao-d:D_1N4148_T4 D?
+L taobao-d:D_1N4148_T4 D2
 U 1 1 5CF7436F
 P 3150 1800
-F 0 "D?" H 3150 2050 50  0000 C CNN
+F 0 "D2" H 3150 2050 50  0000 C CNN
 F 1 "D_1N4148_T4" H 3150 1950 50  0000 C CNN
 F 2 "Diode_SMD:D_SOD-123" V 3150 1800 50  0001 C CNN
@@
 	2650 1800 2850 1800
 $Comp
-L taobao-r:R122,0603 R?
+L taobao-r:R122,0603 R2
 U 1 1 5CF75167
 P 3600 2300
-F 0 "R?" V 3350 2300 50  0000 C CNN
+F 0 "R2" V 3350 2300 50  0000 C CNN
 F 1 "R122,0603" V 3450 2300 50  0000 C CNN
 F 2 "Resistor_SMD:R_0603_1608Metric_Pad1.05x0.95mm_HandSolder" H 3600 2300 50  0001 C CNN
@@
 $EndComp
 $Comp
-L taobao-r:R122,0603 R?
+L taobao-r:R122,0603 R3
 U 1 1 5CF75A58
 P 3600 2550
-F 0 "R?" V 3350 2550 50  0000 C CNN
+F 0 "R3" V 3350 2550 50  0000 C CNN
 F 1 "R122,0603" V 3450 2550 50  0000 C CNN
 F 2 "Resistor_SMD:R_0603_1608Metric_Pad1.05x0.95mm_HandSolder" H 3600 2550 50  0001 C CNN
@@
 $EndComp
 $Comp
-L taobao-r:R122,0603 R?
+L taobao-r:R122,0603 R5
 U 1 1 5CF75C3A
 P 3600 2850
-F 0 "R?" V 3350 2850 50  0000 C CNN
+F 0 "R5" V 3350 2850 50  0000 C CNN
 F 1 "R122,0603" V 3450 2850 50  0000 C CNN
 F 2 "Resistor_SMD:R_0603_1608Metric_Pad1.05x0.95mm_HandSolder" H 3600 2850 50  0001 C CNN
@@
 $EndComp
 $Comp
-L taobao-led:LED_RED,0603 D?
+L taobao-led:LED_RED,0603 D5
 U 1 1 5CF768BE
 P 3200 2850
-F 0 "D?" H 3200 2600 50  0000 C CNN
+F 0 "D5" H 3200 2600 50  0000 C CNN
 F 1 "LED_RED,0603" H 3200 2700 50  0000 C CNN
 F 2 "footprint-lib:LED_0603_1608Metric" V 3200 2850 50  0001 C CNN
@@
 $EndComp
 $Comp
-L taobao-led:LED_GREEN,0603 D?
+L taobao-led:LED_GREEN,0603 D4
 U 1 1 5CF7747C
 P 3200 2550
-F 0 "D?" H 3200 2300 50  0000 C CNN
+F 0 "D4" H 3200 2300 50  0000 C CNN
 F 1 "LED_GREEN,0603" H 3200 2400 50  0000 C CNN
 F 2 "footprint-lib:LED_0603_1608Metric" V 3200 2550 50  0001 C CNN
@@
 $EndComp
 $Comp
-L taobao-led:LED_ORANGE,0603 D?
+L taobao-led:LED_ORANGE,0603 D3
 U 1 1 5CF77A82
 P 3200 2300
-F 0 "D?" H 3200 2050 50  0000 C CNN
+F 0 "D3" H 3200 2050 50  0000 C CNN
 F 1 "LED_ORANGE,0603" H 3200 2150 50  0000 C CNN
 F 2 "footprint-lib:LED_0603_1608Metric" V 3200 2300 50  0001 C CNN
@@
 Connection ~ 2850 2550
 $Comp
-L taobao-components:USB_Micro U?
+L taobao-components:USB_Micro U1
 U 1 1 5CF7C2FA
 P 1250 2200
-F 0 "U?" H 1250 2700 50  0000 C CNN
+F 0 "U1" H 1250 2700 50  0000 C CNN
 F 1 "USB_Micro" H 1250 2600 50  0000 C CNN
 F 2 "footprint-lib:USB_Micro-B_Molex-105017-0001" H 1250 1700 50  0001 C CNN
@@
 	1800 2000 3950 2000
 $Comp
-L power:GND #PWR?
+L power:GND #PWR0103
 U 1 1 5CF7E46F
 P 1800 2500
-F 0 "#PWR?" H 1800 2250 50  0001 C CNN
+F 0 "#PWR0103" H 1800 2250 50  0001 C CNN
 F 1 "GND" H 1850 2300 50  0000 C CNN
 F 2 "" H 1800 2500 50  0001 C CNN
@@
 	1800 2400 1800 2500
 $Comp
-L power:GND #PWR?
+L power:GND #PWR0104
 U 1 1 5CF7EB3B
 P 750 2550
-F 0 "#PWR?" H 750 2300 50  0001 C CNN
+F 0 "#PWR0104" H 750 2300 50  0001 C CNN
 F 1 "GND" H 800 2350 50  0000 C CNN
 F 2 "" H 750 2550 50  0001 C CNN
@@
 $EndComp
 Wire Wire Line
-	750  2550 750  2300
+	750  2550 750  2400
 Wire Wire Line
 	750  2000 850  2000
@@
 Connection ~ 750  2300
 Wire Wire Line
-	750  2300 750  2000
+	750  2300 750  2100
 Wire Wire Line
 	850  2400 750  2400
 $Comp
-L taobao-r:R103,0603 R?
+L taobao-r:R103,0603 R1
 U 1 1 5CF7FBAA
 P 5900 2250
-F 0 "R?" V 5650 2250 50  0000 C CNN
+F 0 "R1" V 5650 2250 50  0000 C CNN
 F 1 "R103,0603" V 5750 2250 50  0000 C CNN
 F 2 "Resistor_SMD:R_0603_1608Metric_Pad1.05x0.95mm_HandSolder" H 5900 2250 50  0001 C CNN
@@
 $EndComp
 $Comp
-L taobao-r:R122,0603 R?
+L taobao-r:R122,0603 R4
 U 1 1 5CF80BC3
 P 5900 2600
-F 0 "R?" V 5650 2600 50  0000 C CNN
+F 0 "R4" V 5650 2600 50  0000 C CNN
 F 1 "R122,0603" V 5750 2600 50  0000 C CNN
 F 2 "Resistor_SMD:R_0603_1608Metric_Pad1.05x0.95mm_HandSolder" H 5900 2600 50  0001 C CNN
@@
 $EndComp
 $Comp
-L power:GND #PWR?
+L power:GND #PWR0105
 U 1 1 5CF83AAD
 P 6250 3350
-F 0 "#PWR?" H 6250 3100 50  0001 C CNN
+F 0 "#PWR0105" H 6250 3100 50  0001 C CNN
 F 1 "GND" H 6300 3150 50  0000 C CNN
 F 2 "" H 6250 3350 50  0001 C CNN
@@
 Connection ~ 6250 2600
 $Comp
-L Device:Fuse_Small F?
+L Device:Fuse_Small F1
 U 1 1 5CF8671F
 P 6050 1900
-F 0 "F?" H 6050 2100 50  0000 C CNN
-F 1 "Fuse_Small" H 6050 2000 50  0000 C CNN
-F 2 "" H 6050 1900 50  0001 C CNN
+F 0 "F1" H 6050 2100 50  0000 C CNN
+F 1 "Fuse_Small,0805" H 6050 2000 50  0000 C CNN
+F 2 "Resistor_SMD:R_0805_2012Metric_Pad1.15x1.40mm_HandSolder" H 6050 1900 50  0001 C CNN
 F 3 "~" H 6050 1900 50  0001 C CNN
 	1    6050 1900
@@
 Wire Wire Line
 	5550 1900 5950 1900
-$Comp
-L taobao-cp:CP47uf,16V C?
-U 1 1 5CF885DE
-P 6550 2200
-F 0 "C?" H 6650 2250 50  0000 L CNN
-F 1 "CP47uf,16V" H 6650 2200 50  0000 L CNN
-F 2 "Capacitor_SMD:CP_Elec_5x5.3" H 6550 2200 50  0001 C CNN
-F 3 "~" H 6550 2200 50  0001 C CNN
-	1    6550 2200
-	1    0    0    -1
-$EndComp
 Wire Wire Line
 	6150 1900 6550 1900
@@
 	6550 1900 6550 2100
 $Comp
-L power:GND #PWR?
+L power:GND #PWR0106
 U 1 1 5CF891FE
 P 6550 3350
-F 0 "#PWR?" H 6550 3100 50  0001 C CNN
+F 0 "#PWR0106" H 6550 3100 50  0001 C CNN
 F 1 "GND" H 6600 3150 50  0000 C CNN
 F 2 "" H 6550 3350 50  0001 C CNN
@@
 	6550 2300 6550 3350
 $Comp
-L my_power:Vout #PWR?
+L my_power:Vout #PWR0107
 U 1 1 5CF89FC6
 P 7000 1750
-F 0 "#PWR?" H 7000 1600 50  0001 C CNN
+F 0 "#PWR0107" H 7000 1600 50  0001 C CNN
 F 1 "Vout" H 7050 1900 50  0000 C CNN
 F 2 "" H 7000 1750 50  0001 C CNN
@@
 	7000 1900 6550 1900
 Connection ~ 6550 1900
+NoConn ~ 1650 2100
+NoConn ~ 1650 2200
+NoConn ~ 1650 2300
+Connection ~ 750  2100
+Wire Wire Line
+	750  2100 750  2000
+Connection ~ 750  2400
+Wire Wire Line
+	750  2400 750  2300
+$Comp
+L taobao-c:C106,0805 C1
+U 1 1 5D067E4E
+P 6550 2200
+F 0 "C1" H 6650 2250 50  0000 L CNN
+F 1 "C106,0805" H 6650 2200 50  0000 L CNN
+F 2 "Capacitor_SMD:C_0805_2012Metric_Pad1.15x1.40mm_HandSolder" H 6550 2200 50  0001 C CNN
+F 3 "~" H 6550 2200 50  0001 C CNN
+	1    6550 2200
+	1    0    0    -1
+$EndComp
 $EndSCHEMATC
