File: hardware/MCP73837.sch (KiCad schematic (older format))
At the start: 14 parts, among them U1 USB_Micro, U2 MCP73837_MSOP10

Commit message: update filename,
Parts:
- removed C1: CP47uf,16V, Capacitor_SMD:CP_Elec_5x5.3, symbol taobao-cp:CP47uf,16V
- added C1: C106,0805, Capacitor_SMD:C_0805_2012Metric_Pad1.15x1.40mm_HandSolder, symbol taobao-c:C106,0805
- added J?: OUT_HEADER, symbol Connector:Conn_01x03_Female
Connections:
- net GND: now also C1.2, J?.1 (Pin_1)
- net Vout: now also C1.1, J?.2 (Pin_2)
Changed lines of the file:
@@
 Wire Wire Line
 	5550 1900 5950 1900
-$Comp
-L taobao-cp:CP47uf,16V C1
-U 1 1 5CF885DE
-P 6550 2200
-F 0 "C1" H 6650 2250 50  0000 L CNN
-F 1 "CP47uf,16V" H 6650 2200 50  0000 L CNN
-F 2 "Capacitor_SMD:CP_Elec_5x5.3" H 6550 2200 50  0001 C CNN
-F 3 "~" H 6550 2200 50  0001 C CNN
-	1    6550 2200
-	1    0    0    -1
-$EndComp
 Wire Wire Line
 	6150 1900 6550 1900
@@
 Wire Wire Line
 	750  2400 750  2300
+$Comp
+L taobao-c:C106,0805 C1
+U 1 1 5D067E4E
+P 6550 2200
+F 0 "C1" H 6650 2250 50  0000 L CNN
+F 1 "C106,0805" H 6650 2200 50  0000 L CNN
+F 2 "Capacitor_SMD:C_0805_2012Metric_Pad1.15x1.40mm_HandSolder" H 6550 2200 50  0001 C CNN
+F 3 "~" H 6550 2200 50  0001 C CNN
+	1    6550 2200
+	1    0    0    -1
+$EndComp
+$Comp
+L power:GND #PWR?
+U 1 1 5D06EF6A
+P 7100 2850
+F 0 "#PWR?" H 7100 2600 50  0001 C CNN
+F 1 "GND" H 7150 2650 50  0000 C CNN
+F 2 "" H 7100 2850 50  0001 C CNN
+F 3 "" H 7100 2850 50  0001 C CNN
+	1    7100 2850
+	1    0    0    -1
+$EndComp
+$Comp
+L Connector:Conn_01x03_Female J?
+U 1 1 5D06F529
+P 7400 2500
+F 0 "J?" H 7300 2150 50  0000 C CNN
+F 1 "OUT_HEADER" H 7300 2250 50  0000 C CNN
+F 2 "" H 7400 2500 50  0001 C CNN
+F 3 "~" H 7400 2500 50  0001 C CNN
+	1    7400 2500
+	1    0    0    1
+$EndComp
+Wire Wire Line
+	7200 2600 7100 2600
+Wire Wire Line
+	7100 2600 7100 2850
+$Comp
+L my_power:Vout #PWR?
+U 1 1 5D07073C
+P 6950 2850
+F 0 "#PWR?" H 6950 2700 50  0001 C CNN
+F 1 "Vout" H 7000 3000 50  0000 C CNN
+F 2 "" H 6950 2850 50  0001 C CNN
+F 3 "" H 6950 2850 50  0001 C CNN
+	1    6950 2850
+	-1   0    0    1
+$EndComp
+Wire Wire Line
+	6950 2850 6950 2500
+Wire Wire Line
+	6950 2500 7200 2500
 $EndSCHEMATC
